Commit message: fix(urdf): RobotModel render sorunu cozuldu - kok neden: eksik collision+inertial bloklari (RViz/Ogre bazi ortamlarda bunlar olmadan link'leri atliyor)

File: src/ika_bringup/urdf/ika.urdf (robot description, URDF)
Before this commit: robot ika, 10 links, 9 joints
Links:
- link base_link: mass None -> 6.0; geometry collision box size=0.5 0.35 0.15; visual box size=0.5 0.35 0.15
- link gps_link: mass None -> 0.05; geometry collision cylinder length=0.02 radius=0.03; visual cylinder length=0.02 radius=0.03
- link imu_link: mass None -> 0.01; geometry collision box size=0.03 0.03 0.01; visual box size=0.03 0.03 0.01
- link laser_link: mass None -> 0.19; geometry collision cylinder length=0.05 radius=0.04; visual cylinder length=0.05 radius=0.04
- link wheel_fl: mass None -> 0.3; geometry collision cylinder length=0.05 radius=0.065; visual cylinder length=0.05 radius=0.065
- link wheel_fr: mass None -> 0.3; geometry collision cylinder length=0.05 radius=0.065; visual cylinder length=0.05 radius=0.065
- link wheel_ml: mass None -> 0.3; geometry collision cylinder length=0.05 radius=0.065; visual cylinder length=0.05 radius=0.065
- link wheel_mr: mass None -> 0.3; geometry collision cylinder length=0.05 radius=0.065; visual cylinder length=0.05 radius=0.065
- link wheel_rl: mass None -> 0.3; geometry collision cylinder length=0.05 radius=0.065; visual cylinder length=0.05 radius=0.065
- link wheel_rr: mass None -> 0.3; geometry collision cylinder length=0.05 radius=0.065; visual cylinder length=0.05 radius=0.065
